File: kiCAD/Endstops.sch (KiCad schematic (older format))
At the start: 0 parts

Commit message: Completed Schematic, assigned footprints.
Parts:
- added C152, C153, C154, C155, C156, C157: 10n, Capacitor_SMD:C_0603_1608Metric_Pad1.05x0.95mm_HandSolder, symbol Device:C_Small
- added D41, D42, D43, D44, D45, D46: LED_Small, Diode_SMD:D_0603_1608Metric_Pad1.05x0.95mm_HandSolder, symbol Device:LED_Small
- added J28, J29, J30, J31, J32, J33: Conn_01x03, Connector_Molex:Molex_KK-254_AE-6410-03A_1x03_P2.54mm_Vertical, symbol Connector_Generic:Conn_01x03
- added JP10, JP13, JP14, JP17, JP18, JP9: Jumper_3_Open, Connector_PinHeader_2.54mm:PinHeader_1x03_P2.54mm_Vertical, symbol Jumper:Jumper_3_Open
- added JP11, JP12, JP15, JP16, JP7, JP8: SENSORLESS, Connector_PinHeader_2.54mm:PinHeader_1x02_P2.54mm_Vertical, symbol Device:Jumper_NC_Small
- added R80, R81, R84, R85, R88, R89: 10k, Resistor_SMD:R_0603_1608Metric_Pad1.05x0.95mm_HandSolder, symbol Device:R_Small_US
- added R82, R83, R86, R87, R90, R91: 2.2k, Resistor_SMD:R_0603_1608Metric_Pad1.05x0.95mm_HandSolder, symbol Device:R_Small_US
Connections:
- new net: D41.1 (K), J28.1 (Pin_1), R80.1
- new net: J28.2 (Pin_2), JP9.2 (C), R82.2
- new net: D41.2 (A), R82.1
- new net: D43.1 (K), J30.1 (Pin_1), R84.1
- new net: J30.2 (Pin_2), JP13.2 (C), R86.2
- new net: D43.2 (A), R86.1
- new net: D45.1 (K), J32.1 (Pin_1), R88.1
- new net: J32.2 (Pin_2), JP17.2 (C), R90.2
- new net: D45.2 (A), R90.1
- new net: D42.1 (K), J29.1 (Pin_1), R81.1
- new net: J29.2 (Pin_2), JP10.2 (C), R83.2
- new net: D42.2 (A), R83.1
- new net: D44.1 (K), J31.1 (Pin_1), R85.1
- new net: J31.2 (Pin_2), JP14.2 (C), R87.2
- new net: D44.2 (A), R87.1
- new net: D46.1 (K), J33.1 (Pin_1), R89.1
- new net: J33.2 (Pin_2), JP18.2 (C), R91.2
- new net: D46.2 (A), R91.1
- new net +3V3: JP10.3 (B), JP13.3 (B), JP14.3 (B), JP17.3 (B), JP18.3 (B), JP9.3 (B)
- new net +5V: JP10.1 (A), JP13.1 (A), JP14.1 (A), JP17.1 (A), JP18.1 (A), JP9.1 (A)
- new net E0_DIAG: JP8.1
- new net E0_STOP: C153.1, JP8.2, R81.2
- new net E1_DIAG: JP12.1
- new net E1_STOP: C155.1, JP12.2, R85.2
- new net E2_DIAG: JP16.1
- new net E2_STOP: C157.1, JP16.2, R89.2
- new net GND: C152.2, C153.2, C154.2, C155.2, C156.2, C157.2, J28.3 (Pin_3), J29.3 (Pin_3), J30.3 (Pin_3), J31.3 (Pin_3), J32.3 (Pin_3), J33.3 (Pin_3)
- new net X_DIAG: JP7.1
- new net X_STOP: C152.1, JP7.2, R80.2
- new net Y_DIAG: JP11.1
- new net Y_STOP: C154.1, JP11.2, R84.2
- new net Z_DIAG: JP15.1
- new net Z_STOP: C156.1, JP15.2, R88.2
Other:
- note added: "ENDSTOPS\n"
