File: kiCAD/Thermistors.sch (KiCad schematic (older format))
At the start: 0 parts

Commit message: Completed Schematic, assigned footprints.
Parts:
- added C148, C149, C150, C151: 100n, Capacitor_SMD:C_0603_1608Metric_Pad1.05x0.95mm_HandSolder, symbol Device:C_Small
- added D37, D38, D39, D40: BAV99W, Package_TO_SOT_SMD:SOT-323_SC-70_Handsoldering, symbol Device:D_Schottky_x2_Serial_AKC
- added J24, J25, J26, J27: Conn_01x02, Connector_Molex:Molex_KK-254_AE-6410-02A_1x02_P2.54mm_Vertical, symbol Connector_Generic:Conn_01x02
- added R68, R69, R70, R71, R74, R75, R76, R77: 2.37k, Resistor_SMD:R_0603_1608Metric_Pad1.05x0.95mm_HandSolder, symbol Device:R_Small_US
- added R72, R73, R78, R79: 4.7k, Resistor_SMD:R_0603_1608Metric_Pad1.05x0.95mm_HandSolder, symbol Device:R_Small_US
Connections:
- new net: J24.1 (Pin_1), R70.1, R72.2
- new net: D37.3 (common), R68.1, R70.2
- new net: J25.1 (Pin_1), R71.1, R73.2
- new net: D38.3 (common), R69.1, R71.2
- new net: J26.1 (Pin_1), R76.1, R78.2
- new net: D39.3 (common), R74.1, R76.2
- new net: J27.1 (Pin_1), R77.1, R79.2
- new net: D40.3 (common), R75.1, R77.2
- new net +3V3: D37.2 (K), D38.2 (K), D39.2 (K), D40.2 (K), R72.1, R73.1, R78.1, R79.1
- new net GND: C148.2, C149.2, C150.2, C151.2, D37.1 (A), D38.1 (A), D39.1 (A), D40.1 (A), J24.2 (Pin_2), J25.2 (Pin_2), J26.2 (Pin_2), J27.2 (Pin_2)
- new net T0: C148.1, R68.2
- new net T1: C150.1, R74.2
- new net T2: C149.1, R69.2
- new net TB: C151.1, R75.2
Other:
- note added: "THERMISTORS"
