File: kiCAD/_autosave-WorkhorseBoard.kicad_pcb (KiCad board)
At the start: 4 copper layers, 205 x 97 mm, 385 parts, among them J1 USB_B_Mini, J10 MAIN_POWER, J11 BED_POWER, J12 H0, J13 F0, J14 5V_EXT, J15 F1, J16 F4, J17 H1, J19 F2, J2 Micro_SD_Card, J20 F5, J21 H2, J22 F3, J23 HB, J24 Conn_01x02, J25 Conn_01x02, J26 Conn_01x02, J27 Conn_01x02, J28 Conn_01x03, J29 Conn_01x03, J3 Conn_01x06, J30 Conn_01x03, J31 Conn_01x03, J32 Conn_01x03, J33 Conn_01x03, J4 X, J5 E0, J6 Y, J7 E1, J8 Z, J9 E2, Q1 Q_NMOS_GSD, Q10 Q_NMOS_GDS, Q2 Q_NMOS_GDS, Q3 Q_NMOS_GSD, Q4 Q_NMOS_GSD, Q5 Q_NMOS_GDS, Q6 Q_NMOS_GSD, Q7 Q_NMOS_GSD, Q8 Q_NMOS_GDS, Q9 Q_NMOS_GSD, SW1 SW_Push, U1 24C02, U10 TPS54531, U11 TPS54531, U12 AP7361C-33E-13, U13 74HCT365, U14 74HCT365, U2 USBLC6-2SC6, U3 STM32F446VETx, U4 TMC2209, U5 TMC2209, U6 TMC2209, U7 TMC2209, U8 TMC2209, U9 TMC2209, Y1 X322512MSB4SI

Commit message: Re-did fills
Routing:
- net +24V: track 248.9 -> 11.4 mm, vias 0 -> 215
- net VM: track 87.4 -> 35.3 mm, vias 90 -> 102
- net +5V: track 62.3 -> 31.3 mm
- net GND: track 448.6 -> 423.0 mm, vias 2 -> 22
- net +12V: track 20.2 -> 4.99 mm
- added copper zone on F.Cu, net GND
